File: HubController.kicad_sch (KiCad schematic)
At the start: 1 part, among them J2 USB_C_Receptacle

Commit message: start layout of usb PD
Parts:
- removed J2: USB_C_Receptacle, symbol Connector:USB_C_Receptacle
Connections:
- no-connect marks 15 -> 0
Changed lines of the file:
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@@
 (kicad_sch (version 20230121) (generator eeschema)
   (paper "A4")
-  (junction (at 52.832 29.718) (diameter 0) (color 0 0 0 0)
-  )
-  (junction (at 37.084 96.012) (diameter 0) (color 0 0 0 0)
-  )
-  (no_connect (at 52.324 47.498))
-  (no_connect (at 52.324 57.658))
-  (no_connect (at 52.324 80.518))
-  (no_connect (at 52.324 55.118))
-  (no_connect (at 52.324 88.138))
-  (no_connect (at 52.324 42.418))
-  (no_connect (at 29.464 95.758))
-  (no_connect (at 52.324 44.958))
-  (no_connect (at 52.324 62.738))
-  (no_connect (at 52.324 70.358))
-  (no_connect (at 52.324 72.898))
-  (no_connect (at 52.324 65.278))
-  (no_connect (at 52.324 50.038))
-  (no_connect (at 52.324 85.598))
-  (no_connect (at 52.324 77.978))
-  (wire (pts (xy 54.61 29.718) (xy 52.832 29.718))
-    (stroke (width 0) (type default))
-  )
-  (wire (pts (xy 37.084 95.758) (xy 37.084 96.012))
-    (stroke (width 0) (type default))
-  )
-  (wire (pts (xy 52.832 29.718) (xy 52.324 29.718))
-    (stroke (width 0) (type default))
-  )
-  (wire (pts (xy 37.084 96.012) (xy 37.084 97.536))
-    (stroke (width 0) (type default))
-  )
-  (wire (pts (xy 55.118 37.338) (xy 52.324 37.338))
-    (stroke (width 0) (type default))
-  )
-  (wire (pts (xy 55.118 34.798) (xy 52.324 34.798))
-    (stroke (width 0) (type default))
-  )
-  (global_label "USB_UFP_CC1" (shape input) (at 55.118 34.798 0) (fields_autoplaced)
-    (effects (font (size 1.27 1.27)) (justify left))
-    (property "Intersheetrefs" "${INTERSHEET_REFS}" (at 71.287 34.798 0)
-      (effects (font (size 1.27 1.27)) (justify left) hide)
-    )
-  )
-  (global_label "USB_UFP_CC2" (shape input) (at 55.118 37.338 0) (fields_autoplaced)
-    (effects (font (size 1.27 1.27)) (justify left))
-    (property "Intersheetrefs" "${INTERSHEET_REFS}" (at 71.287 37.338 0)
-      (effects (font (size 1.27 1.27)) (justify left) hide)
-    )
-  )
-  (global_label "VBUS" (shape input) (at 54.61 29.718 0) (fields_autoplaced)
-    (effects (font (size 1.27 1.27)) (justify left))
-    (property "Intersheetrefs" "${INTERSHEET_REFS}" (at 62.4938 29.718 0)
-      (effects (font (size 1.27 1.27)) (justify left) hide)
-    )
-  )
-  (symbol (lib_id "Connector:USB_C_Receptacle") (at 37.084 55.118 0) (unit 1)
-    (in_bom yes) (on_board yes) (dnp no) (fields_autoplaced)
-    (property "Reference" "J2" (at 37.084 22.86 0)
-      (effects (font (size 1.27 1.27)))
-    )
-    (property "Value" "USB_C_Receptacle" (at 37.084 25.4 0)
-      (effects (font (size 1.27 1.27)))
-    )
-    (property "Footprint" "" (at 40.894 55.118 0)
-      (effects (font (size 1.27 1.27)) hide)
-    )
-    (property "Datasheet" "https://www.usb.org/sites/default/files/documents/usb_type-c.zip" (at 40.894 55.118 0)
-      (effects (font (size 1.27 1.27)) hide)
-    )
-    (pin "A5")
-    (pin "B2")
-    (pin "B6")
-    (pin "A11")
-    (pin "A3")
-    (pin "B4")
-    (pin "B3")
-    (pin "B5")
-    (pin "B1")
-    (pin "B12")
-    (pin "A1")
-    (pin "B8")
-    (pin "B7")
-    (pin "A6")
-    (pin "A4")
-    (pin "A12")
-    (pin "A2")
-    (pin "A7")
-    (pin "A8")
-    (pin "B11")
-    (pin "S1")
-    (pin "B10")
-    (pin "A9")
-    (pin "A10")
-    (pin "B9")
-    (instances
-      (project "USBHUB"
-        (path "/d5edc647-9ac3-4ac1-ab8a-57c77be3f4d3/521afbfd-a43d-40d3-b71e-52d74f5665e8"
-          (reference "J2") (unit 1)
-        )
-      )
-    )
-  )
-  (symbol (lib_id "power:GND") (at 37.084 97.536 0) (unit 1)
-    (in_bom yes) (on_board yes) (dnp no) (fields_autoplaced)
-    (property "Reference" "#PWR014" (at 37.084 103.886 0)
-      (effects (font (size 1.27 1.27)) hide)
-    )
-    (property "Value" "GND" (at 37.084 102.87 0)
-      (effects (font (size 1.27 1.27)))
-    )
-    (property "Footprint" "" (at 37.084 97.536 0)
-      (effects (font (size 1.27 1.27)) hide)
-    )
-    (property "Datasheet" "" (at 37.084 97.536 0)
-      (effects (font (size 1.27 1.27)) hide)
-    )
-    (pin "1")
-    (instances
-      (project "USBHUB"
-        (path "/d5edc647-9ac3-4ac1-ab8a-57c77be3f4d3/521afbfd-a43d-40d3-b71e-52d74f5665e8"
-          (reference "#PWR014") (unit 1)
-        )
-      )
-    )
-  )
-  (symbol (lib_id "power:PWR_FLAG") (at 52.832 29.718 0) (unit 1)
-    (in_bom yes) (on_board yes) (dnp no) (fields_autoplaced)
-    (property "Reference" "#FLG01" (at 52.832 27.813 0)
-      (effects (font (size 1.27 1.27)) hide)
-    )
-    (property "Value" "PWR_FLAG" (at 52.832 25.4 0)
-      (effects (font (size 1.27 1.27)))
-    )
-    (property "Footprint" "" (at 52.832 29.718 0)
-      (effects (font (size 1.27 1.27)) hide)
-    )
-    (property "Datasheet" "~" (at 52.832 29.718 0)
-      (effects (font (size 1.27 1.27)) hide)
-    )
-    (pin "1")
-    (instances
-      (project "USBHUB"
-        (path "/d5edc647-9ac3-4ac1-ab8a-57c77be3f4d3/521afbfd-a43d-40d3-b71e-52d74f5665e8"
-          (reference "#FLG01") (unit 1)
-        )
-      )
-    )
-  )
-  (symbol (lib_id "power:PWR_FLAG") (at 37.084 96.012 270) (unit 1)
-    (in_bom yes) (on_board yes) (dnp no) (fields_autoplaced)
-    (property "Reference" "#FLG02" (at 38.989 96.012 0)
-      (effects (font (size 1.27 1.27)) hide)
-    )
-    (property "Value" "PWR_FLAG" (at 40.64 96.012 90)
-      (effects (font (size 1.27 1.27)) (justify left))
-    )
-    (property "Footprint" "" (at 37.084 96.012 0)
-      (effects (font (size 1.27 1.27)) hide)
-    )
-    (property "Datasheet" "~" (at 37.084 96.012 0)
-      (effects (font (size 1.27 1.27)) hide)
-    )
-    (pin "1")
-    (instances
-      (project "USBHUB"
-        (path "/d5edc647-9ac3-4ac1-ab8a-57c77be3f4d3/521afbfd-a43d-40d3-b71e-52d74f5665e8"
-          (reference "#FLG02") (unit 1)
-        )
-      )
-    )
-  )
 )

Commit message: fix warnings
Parts:
- added J2: USB_C_Receptacle, symbol Connector:USB_C_Receptacle
Connections:
- new net GND: J2.A1 (GND), J2.A12 (GND), J2.B1 (GND), J2.B12 (GND)
- new net USB_UFP_CC1: J2.A5 (CC1)
- new net USB_UFP_CC2: J2.B5 (CC2)
- new net VBUS: J2.A4 (VBUS), J2.A9 (VBUS), J2.B4 (VBUS), J2.B9 (VBUS)
- no-connect marks 0 -> 15
Changed lines of the file:
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@@
 (kicad_sch (version 20230121) (generator eeschema)
   (paper "A4")
+  (junction (at 52.832 29.718) (diameter 0) (color 0 0 0 0)
+  )
+  (junction (at 37.084 96.012) (diameter 0) (color 0 0 0 0)
+  )
+  (no_connect (at 52.324 47.498))
+  (no_connect (at 52.324 57.658))
+  (no_connect (at 52.324 80.518))
+  (no_connect (at 52.324 55.118))
+  (no_connect (at 52.324 88.138))
+  (no_connect (at 52.324 42.418))
+  (no_connect (at 29.464 95.758))
+  (no_connect (at 52.324 44.958))
+  (no_connect (at 52.324 62.738))
+  (no_connect (at 52.324 70.358))
+  (no_connect (at 52.324 72.898))
+  (no_connect (at 52.324 65.278))
+  (no_connect (at 52.324 50.038))
+  (no_connect (at 52.324 85.598))
+  (no_connect (at 52.324 77.978))
+  (wire (pts (xy 54.61 29.718) (xy 52.832 29.718))
+    (stroke (width 0) (type default))
+  )
+  (wire (pts (xy 37.084 95.758) (xy 37.084 96.012))
+    (stroke (width 0) (type default))
+  )
+  (wire (pts (xy 52.832 29.718) (xy 52.324 29.718))
+    (stroke (width 0) (type default))
+  )
+  (wire (pts (xy 37.084 96.012) (xy 37.084 97.536))
+    (stroke (width 0) (type default))
+  )
+  (wire (pts (xy 55.118 37.338) (xy 52.324 37.338))
+    (stroke (width 0) (type default))
+  )
+  (wire (pts (xy 55.118 34.798) (xy 52.324 34.798))
+    (stroke (width 0) (type default))
+  )
+  (global_label "USB_UFP_CC1" (shape input) (at 55.118 34.798 0) (fields_autoplaced)
+    (effects (font (size 1.27 1.27)) (justify left))
+    (property "Intersheetrefs" "${INTERSHEET_REFS}" (at 71.287 34.798 0)
+      (effects (font (size 1.27 1.27)) (justify left) hide)
+    )
+  )
+  (global_label "USB_UFP_CC2" (shape input) (at 55.118 37.338 0) (fields_autoplaced)
+    (effects (font (size 1.27 1.27)) (justify left))
+    (property "Intersheetrefs" "${INTERSHEET_REFS}" (at 71.287 37.338 0)
+      (effects (font (size 1.27 1.27)) (justify left) hide)
+    )
+  )
+  (global_label "VBUS" (shape input) (at 54.61 29.718 0) (fields_autoplaced)
+    (effects (font (size 1.27 1.27)) (justify left))
+    (property "Intersheetrefs" "${INTERSHEET_REFS}" (at 62.4938 29.718 0)
+      (effects (font (size 1.27 1.27)) (justify left) hide)
+    )
+  )
+  (symbol (lib_id "Connector:USB_C_Receptacle") (at 37.084 55.118 0) (unit 1)
+    (in_bom yes) (on_board yes) (dnp no) (fields_autoplaced)
+    (property "Reference" "J2" (at 37.084 22.86 0)
+      (effects (font (size 1.27 1.27)))
+    )
+    (property "Value" "USB_C_Receptacle" (at 37.084 25.4 0)
+      (effects (font (size 1.27 1.27)))
+    )
+    (property "Footprint" "" (at 40.894 55.118 0)
+      (effects (font (size 1.27 1.27)) hide)
+    )
+    (property "Datasheet" "https://www.usb.org/sites/default/files/documents/usb_type-c.zip" (at 40.894 55.118 0)
+      (effects (font (size 1.27 1.27)) hide)
+    )
+    (pin "A5")
+    (pin "B2")
+    (pin "B6")
+    (pin "A11")
+    (pin "A3")
+    (pin "B4")
+    (pin "B3")
+    (pin "B5")
+    (pin "B1")
+    (pin "B12")
+    (pin "A1")
+    (pin "B8")
+    (pin "B7")
+    (pin "A6")
+    (pin "A4")
+    (pin "A12")
+    (pin "A2")
+    (pin "A7")
+    (pin "A8")
+    (pin "B11")
+    (pin "S1")
+    (pin "B10")
+    (pin "A9")
+    (pin "A10")
+    (pin "B9")
+    (instances
+      (project "USBHUB"
+        (path "/d5edc647-9ac3-4ac1-ab8a-57c77be3f4d3/521afbfd-a43d-40d3-b71e-52d74f5665e8"
+          (reference "J2") (unit 1)
+        )
+      )
+    )
+  )
+  (symbol (lib_id "power:GND") (at 37.084 97.536 0) (unit 1)
+    (in_bom yes) (on_board yes) (dnp no) (fields_autoplaced)
+    (property "Reference" "#PWR014" (at 37.084 103.886 0)
+      (effects (font (size 1.27 1.27)) hide)
+    )
+    (property "Value" "GND" (at 37.084 102.87 0)
+      (effects (font (size 1.27 1.27)))
+    )
+    (property "Footprint" "" (at 37.084 97.536 0)
+      (effects (font (size 1.27 1.27)) hide)
+    )
+    (property "Datasheet" "" (at 37.084 97.536 0)
+      (effects (font (size 1.27 1.27)) hide)
+    )
+    (pin "1")
+    (instances
+      (project "USBHUB"
+        (path "/d5edc647-9ac3-4ac1-ab8a-57c77be3f4d3/521afbfd-a43d-40d3-b71e-52d74f5665e8"
+          (reference "#PWR014") (unit 1)
+        )
+      )
+    )
+  )
+  (symbol (lib_id "power:PWR_FLAG") (at 52.832 29.718 0) (unit 1)
+    (in_bom yes) (on_board yes) (dnp no) (fields_autoplaced)
+    (property "Reference" "#FLG01" (at 52.832 27.813 0)
+      (effects (font (size 1.27 1.27)) hide)
+    )
+    (property "Value" "PWR_FLAG" (at 52.832 25.4 0)
+      (effects (font (size 1.27 1.27)))
+    )
+    (property "Footprint" "" (at 52.832 29.718 0)
+      (effects (font (size 1.27 1.27)) hide)
+    )
+    (property "Datasheet" "~" (at 52.832 29.718 0)
+      (effects (font (size 1.27 1.27)) hide)
+    )
+    (pin "1")
+    (instances
+      (project "USBHUB"
+        (path "/d5edc647-9ac3-4ac1-ab8a-57c77be3f4d3/521afbfd-a43d-40d3-b71e-52d74f5665e8"
+          (reference "#FLG01") (unit 1)
+        )
+      )
+    )
+  )
+  (symbol (lib_id "power:PWR_FLAG") (at 37.084 96.012 270) (unit 1)
+    (in_bom yes) (on_board yes) (dnp no) (fields_autoplaced)
+    (property "Reference" "#FLG02" (at 38.989 96.012 0)
+      (effects (font (size 1.27 1.27)) hide)
+    )
+    (property "Value" "PWR_FLAG" (at 40.64 96.012 90)
+      (effects (font (size 1.27 1.27)) (justify left))
+    )
+    (property "Footprint" "" (at 37.084 96.012 0)
+      (effects (font (size 1.27 1.27)) hide)
+    )
+    (property "Datasheet" "~" (at 37.084 96.012 0)
+      (effects (font (size 1.27 1.27)) hide)
+    )
+    (pin "1")
+    (instances
+      (project "USBHUB"
+        (path "/d5edc647-9ac3-4ac1-ab8a-57c77be3f4d3/521afbfd-a43d-40d3-b71e-52d74f5665e8"
+          (reference "#FLG02") (unit 1)
+        )
+      )
+    )
+  )
 )
