File: USBHUB.kicad_pcb (KiCad board)
At the start: 2 copper layers, 24 parts, among them J1 Screw_Terminal_01x02, J2 USB_C_Receptacle, Q1 SI3421DV, Q2 SI3421DV, U1 CYPD3177_24x

Commit message: Finish PCB design
Parts:
- added C8: 3u3, Capacitor_SMD:C_0603_1608Metric, F.Cu at (73.0, 78.5)
- moved R10 15.3 mm to (64.5, 81.2), turned to 0 degrees
- moved R8 11.4 mm to (53.5, 78.0), turned to 180 degrees
- moved R7 5.02 mm to (61.8, 78.5), turned to -90 degrees
- moved D2 3.54 mm to (55.8, 78.8), turned to -90 degrees
- moved R9 3.00 mm to (64.5, 82.8)
- moved J1 2.92 mm to (80.2, 87.0)
- moved C3 1.60 mm to (55.0, 89.6)
- moved R4 1.12 mm to (58.8, 78.5)
- moved R5 1.12 mm to (57.2, 78.5)
- moved R6 1.12 mm to (60.2, 78.5)
- moved C1 0.75 mm to (68.2, 86.1)
- moved C2 0.75 mm to (72.2, 80.2)
- moved D1 0.75 mm to (69.5, 83.0)
- moved Q1 0.75 mm to (72.0, 87.1)
- moved Q2 0.75 mm to (72.5, 83.2)
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Connections:
- J1 pad 1: +20V -> GND
- J1 pad 2: GND -> +20V
- U1 pad 10: USB_UFP_FLIP -> unconnected-(U1-FLIP-Pad10)
Routing:
- net /USB_PD_VDDD_3V3: track 0.00 -> 26.0 mm, vias 0 -> 3
- net +20V: track 0.00 -> 18.3 mm, vias 0 -> 2
- net Net-(D1-A): track 8.83 -> 23.9 mm, vias 0 -> 2
- net GND: track 0.00 -> 11.3 mm, vias 0 -> 20
- net /FAULT: track 0.00 -> 7.12 mm, vias 0 -> 2
- net Net-(U1-ISNK_COARSE): track 0.00 -> 6.76 mm, vias 0 -> 2
- net Net-(U1-HPI_SCL): track 0.00 -> 4.24 mm
- net Net-(U1-HPI_SDA): track 0.00 -> 3.25 mm
- net Net-(U1-ISNK_FINE): track 0.00 -> 3.19 mm
- net Net-(U1-VBUS_FET_EN): track 0.00 -> 2.78 mm
- net Net-(U1-VCCD): track 0.00 -> 2.55 mm
- net Net-(D1-K): track 4.21 -> 6.70 mm
- net Net-(U1-HPI_INT): track 0.00 -> 2.46 mm
- net VBUS: track 23.2 -> 24.7 mm, vias 3 -> 13
- net Net-(D2-K): track 0.00 -> 1.44 mm
- added copper zone on F.Cu, net +20V
- added copper zone on B.Cu, net GND
- added copper zone on F.Cu, net GND
- added copper zone on B.Cu, net VBUS
- added copper zone on F.Cu, net VBUS
Other:
- board outline added: 38.8 x 16.5 mm

Commit message: some touchups
Parts:
- moved D2 0.25 mm to (55.8, 78.5)
Routing:
- net GND: track 11.3 -> 11.6 mm, vias 20 -> 22
Other:
- board text added: "20V/3A USB PD V1.0"
- board text added: "FAULT"
Changed lines of the file:
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@@
   )
   (footprint "LED_SMD:LED_0603_1608Metric" (layer "F.Cu")
-    (at 55.75 78.75 -90)
+    (at 55.75 78.5 -90)
     (descr "LED SMD 0603 (1608 Metric), square (rectangular) end terminal, IPC_7351 nominal, (Body size source: http://www.tortai-tech.com/upload/download/2011102023233369053.pdf), generated with kicad-footprint-generator")
     (tags "LED")
@@
   (gr_arc (start 84.25 91.5) (mid 83.957107 92.207107) (end 83.25 92.5)
     (stroke (width 0.1) (type default)) (layer "Edge.Cuts"))
+  (gr_text "FAULT" (at 58 78) (layer "B.SilkS")
+    (effects (font (size 1 1) (thickness 0.15)) (justify left bottom mirror))
+  )
+  (gr_text "20V/3A USB PD\nV1.0" (at 83.5 79.25) (layer "B.SilkS")
+    (effects (font (size 1 1) (thickness 0.15)) (justify left bottom mirror))
+  )
   (segment (start 56.25 85) (end 57.05 85) (width 0.3) (layer "F.Cu") (net 1))
   (segment (start 53.5 82.75) (end 53.51538 82.75) (width 0.3) (layer "F.Cu") (net 1))
@@
   (segment (start 49.75 87.5) (end 49.5 87.75) (width 0.3) (layer "F.Cu") (net 4))
   (segment (start 58 84.775) (end 58 84.75) (width 0.2) (layer "F.Cu") (net 4))
+  (segment (start 57.775 85.725) (end 57.775 85) (width 0.3) (layer "F.Cu") (net 4))
   (segment (start 58.025 84.75) (end 57.775 85) (width 0.2) (layer "F.Cu") (net 4))
   (segment (start 57.775 87.05) (end 57.975 87.25) (width 0.3) (layer "F.Cu") (net 4))
@@
   (segment (start 49.75 87) (end 49.75 87.5) (width 0.3) (layer "F.Cu") (net 4))
   (segment (start 58 84.75) (end 58.025 84.75) (width 0.2) (layer "F.Cu") (net 4))
+  (segment (start 57.775 85) (end 57.99375 84.78125) (width 0.3) (layer "F.Cu") (net 4))
   (segment (start 59.275 84.875) (end 59 84.75) (width 0.3) (layer "F.Cu") (net 4))
   (segment (start 59 84.75) (end 59.36875 84.78125) (width 0.3) (layer "F.Cu") (net 4))
   (segment (start 51.41 87) (end 51.41 87.41) (width 0.3) (layer "F.Cu") (net 4))
   (segment (start 59.275 85.725) (end 59.275 84.875) (width 0.3) (layer "F.Cu") (net 4))
-  (segment (start 57.775 85) (end 57.775 85.725) (width 0.2) (layer "F.Cu") (net 4))
   (segment (start 49.75 80.75) (end 49.5 80.5) (width 0.3) (layer "F.Cu") (net 4))
   (segment (start 57.975 87.25) (end 57.975 88.75) (width 0.3) (layer "F.Cu") (net 4))
   (segment (start 57.975 88.75) (end 57.975 90.25) (width 0.3) (layer "F.Cu") (net 4))
   (segment (start 49.75 81.5) (end 49.75 80.75) (width 0.3) (layer "F.Cu") (net 4))
+  (via (at 50.5 91) (size 0.7) (drill 0.3) (layers "F.Cu" "B.Cu") (free) (net 4))
   (via (at 58 83.75) (size 0.7) (drill 0.3) (layers "F.Cu" "B.Cu") (net 4))
   (via (at 60 82.75) (size 0.7) (drill 0.3) (layers "F.Cu" "B.Cu") (net 4))
   (via (at 48.75 89.25) (size 0.7) (drill 0.3) (layers "F.Cu" "B.Cu") (free) (net 4))
+  (via (at 50.5 78) (size 0.7) (drill 0.3) (layers "F.Cu" "B.Cu") (free) (net 4))
   (via (at 68 80) (size 0.7) (drill 0.3) (layers "F.Cu" "B.Cu") (free) (net 4))
   (via (at 65 77) (size 0.7) (drill 0.3) (layers "F.Cu" "B.Cu") (free) (net 4))
@@
   (segment (start 70.8625 85.6125) (end 70.8625 86.1625) (width 0.5) (layer "F.Cu") (net 6))
   (segment (start 70.75 85.1875) (end 70.75 85.5) (width 0.5) (layer "F.Cu") (net 6))
-  (segment (start 54.325 78) (end 55.7125 78) (width 0.5) (layer "F.Cu") (net 7))
-  (segment (start 55.7125 78) (end 55.75 77.9625) (width 0.5) (layer "F.Cu") (net 7))
+  (segment (start 54.325 78) (end 55.4625 78) (width 0.3) (layer "F.Cu") (net 7))
+  (segment (start 55.4625 78) (end 55.75 77.7125) (width 0.3) (layer "F.Cu") (net 7))
   (segment (start 55.75 84.25) (end 56.5 83.5) (width 0.3) (layer "F.Cu") (net 10))
   (segment (start 56.5 83.5) (end 57.05 83.5) (width 0.3) (layer "F.Cu") (net 10))
@@
   (segment (start 62.75 84.25) (end 63.675 84.25) (width 0.3) (layer "F.Cu") (net 25))
   (segment (start 62.5 84) (end 62.75 84.25) (width 0.3) (layer "F.Cu") (net 25))
-  (segment (start 58.175 79.825) (end 58.675 79.825) (width 0.25) (layer "F.Cu") (net 26))
-  (segment (start 57.775 80.225) (end 58.175 79.825) (width 0.25) (layer "F.Cu") (net 26))
-  (segment (start 58.675 79.825) (end 58.75 79.75) (width 0.25) (layer "F.Cu") (net 26))
-  (segment (start 58.75 79.75) (end 58.75 79.325) (width 0.25) (layer "F.Cu") (net 26))
+  (segment (start 58.675 79.325) (end 58.75 79.325) (width 0.3) (layer "F.Cu") (net 26))
   (segment (start 58.675 79.4) (end 58.75 79.325) (width 0.2) (layer "F.Cu") (net 26))
-  (segment (start 57.775 80.808358) (end 57.775 80.225) (width 0.25) (layer "F.Cu") (net 26))
-  (segment (start 57.775 81.775) (end 57.775 80.808358) (width 0.3) (layer "F.Cu") (net 26))
+  (segment (start 57.775 81.775) (end 57.775 80.225) (width 0.3) (layer "F.Cu") (net 26))
+  (segment (start 57.775 80.225) (end 58.675 79.325) (width 0.3) (layer "F.Cu") (net 26))
   (segment (start 57.05 82.5) (end 56.5 82.5) (width 0.3) (layer "F.Cu") (net 27))
   (segment (start 57.25 80.5) (end 57.25 79.325) (width 0.3) (layer "F.Cu") (net 27))
@@
   (segment (start 63.875 79.725) (end 63.875 83.625) (width 0.3) (layer "B.Cu") (net 37))
   (segment (start 60.5 87.75) (end 60.5 87) (width 0.3) (layer "B.Cu") (net 37))
+  (segment (start 56.25 80.5) (end 56.25 79.7875) (width 0.25) (layer "F.Cu") (net 38))
   (segment (start 59.5 80.75) (end 59.5 81) (width 0.2) (layer "F.Cu") (net 38))
   (segment (start 59.275 81.225) (end 59.5 80.75) (width 0.2) (layer "F.Cu") (net 38))
-  (segment (start 56.25 80.0375) (end 55.75 79.5375) (width 0.25) (layer "F.Cu") (net 38))
+  (segment (start 56.25 79.7875) (end 55.75 79.2875) (width 0.25) (layer "F.Cu") (net 38))
   (segment (start 59.275 81.775) (end 59.275 81.225) (width 0.2) (layer "F.Cu") (net 38))
-  (segment (start 56.25 80.5) (end 56.25 80.0375) (width 0.25) (layer "F.Cu") (net 38))
   (via (at 59.5 80.75) (size 0.7) (drill 0.3) (layers "F.Cu" "B.Cu") (net 38))
   (via (at 56.25 80.5) (size 0.7) (drill 0.3) (layers "F.Cu" "B.Cu") (net 38))

Commit message: add manufacturing files
Routing:
- net +20V: track 18.3 -> 20.5 mm
Other:
- board text added: "20V"
- board text added: "GND"
Changed lines of the file:
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@@
       (usegerberattributes true)
       (usegerberadvancedattributes true)
-      (creategerberjobfile true)
+      (creategerberjobfile false)
       (dashed_line_dash_ratio 12.000000)
       (dashed_line_gap_ratio 3.000000)
@@
       (outputformat 1)
       (mirror false)
-      (drillshape 1)
+      (drillshape 0)
       (scaleselection 1)
-      (outputdirectory "")
+      (outputdirectory "Manufacturing/")
     )
   )
@@
     (effects (font (size 1 1) (thickness 0.15)) (justify left bottom mirror))
   )
+  (gr_text "GND" (at 83.75 85.5 90) (layer "B.SilkS")
+    (effects (font (size 1 1) (thickness 0.15)) (justify left bottom mirror))
+  )
+  (gr_text "20V" (at 83.75 80.5 90) (layer "B.SilkS")
+    (effects (font (size 1 1) (thickness 0.15)) (justify left bottom mirror))
+  )
   (segment (start 56.25 85) (end 57.05 85) (width 0.3) (layer "F.Cu") (net 1))
   (segment (start 53.5 82.75) (end 53.51538 82.75) (width 0.3) (layer "F.Cu") (net 1))
@@
   (segment (start 58.5 81) (end 58.50137 81) (width 0.25) (layer "F.Cu") (net 3))
   (segment (start 73.025 79.525) (end 73.025 80.25) (width 0.3) (layer "F.Cu") (net 3))
+  (segment (start 72.5 82.1125) (end 72.5 84.3875) (width 0.5) (layer "F.Cu") (net 3))
   (segment (start 72.25 78.75) (end 73.025 79.525) (width 0.3) (layer "F.Cu") (net 3))
   (segment (start 63 80.25) (end 64.75 78.5) (width 0.3) (layer "F.Cu") (net 3))
