File: 01a_VoltageRegulators.kicad_sch (KiCad schematic)
At the start: 34 parts, among them U2 TPS54331, U3 TLV75733PDBV, U4 TPS56637RPAR

Commit message: route power delivery controller
Parts:
- renumbered R12 to R13, R13 to R14, R14 to R15, R15 to R16, R16 to R17, R17 to R18, R18 to R19, R19 to R20, R20 to R21, R21 to R22
Changed lines of the file:
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@@
   (symbol (lib_id "Device:R") (at 138.43 125.73 0) (unit 1)
     (in_bom yes) (on_board yes) (dnp no) (fields_autoplaced)
-    (property "Reference" "R20" (at 140.97 124.46 0)
+    (property "Reference" "R21" (at 140.97 124.46 0)
       (effects (font (size 1.27 1.27)) (justify left))
     )
@@
       (project "USBHUB"
         (path "/d5edc647-9ac3-4ac1-ab8a-57c77be3f4d3/2bd96af5-5a66-4797-badd-32cacbbf4fbd/38e014e7-3281-4b3d-a8ed-ec581f581dff"
-          (reference "R20") (unit 1)
+          (reference "R21") (unit 1)
         )
       )
@@
   (symbol (lib_id "Device:R") (at 34.29 176.53 0) (unit 1)
     (in_bom yes) (on_board yes) (dnp no) (fields_autoplaced)
-    (property "Reference" "R21" (at 36.576 175.26 0)
+    (property "Reference" "R22" (at 36.576 175.26 0)
       (effects (font (size 1.27 1.27)) (justify left))
     )
@@
       (project "USBHUB"
         (path "/d5edc647-9ac3-4ac1-ab8a-57c77be3f4d3/2bd96af5-5a66-4797-badd-32cacbbf4fbd/38e014e7-3281-4b3d-a8ed-ec581f581dff"
-          (reference "R21") (unit 1)
+          (reference "R22") (unit 1)
         )
       )
@@
   (symbol (lib_id "Device:R") (at 134.62 107.95 90) (unit 1)
     (in_bom yes) (on_board yes) (dnp no)
-    (property "Reference" "R18" (at 134.62 102.87 90)
+    (property "Reference" "R19" (at 134.62 102.87 90)
       (effects (font (size 1.27 1.27)))
     )
@@
       (project "USBHUB"
         (path "/d5edc647-9ac3-4ac1-ab8a-57c77be3f4d3/2bd96af5-5a66-4797-badd-32cacbbf4fbd/38e014e7-3281-4b3d-a8ed-ec581f581dff"
-          (reference "R18") (unit 1)
+          (reference "R19") (unit 1)
         )
       )
@@
   (symbol (lib_id "Device:R") (at 110.49 106.68 90) (unit 1)
     (in_bom yes) (on_board yes) (dnp no)
-    (property "Reference" "R16" (at 110.49 101.6 90)
+    (property "Reference" "R17" (at 110.49 101.6 90)
       (effects (font (size 1.27 1.27)))
     )
@@
       (project "USBHUB"
         (path "/d5edc647-9ac3-4ac1-ab8a-57c77be3f4d3/2bd96af5-5a66-4797-badd-32cacbbf4fbd/38e014e7-3281-4b3d-a8ed-ec581f581dff"
-          (reference "R16") (unit 1)
+          (reference "R17") (unit 1)
         )
       )
@@
   (symbol (lib_id "Device:R") (at 152.4 48.26 0) (unit 1)
     (in_bom yes) (on_board yes) (dnp no) (fields_autoplaced)
-    (property "Reference" "R14" (at 154.94 46.99 0)
+    (property "Reference" "R15" (at 154.94 46.99 0)
       (effects (font (size 1.27 1.27)) (justify left))
     )
@@
       (project "USBHUB"
         (path "/d5edc647-9ac3-4ac1-ab8a-57c77be3f4d3/2bd96af5-5a66-4797-badd-32cacbbf4fbd/38e014e7-3281-4b3d-a8ed-ec581f581dff"
-          (reference "R14") (unit 1)
+          (reference "R15") (unit 1)
         )
       )
@@
   (symbol (lib_id "Device:R") (at 127 107.95 90) (unit 1)
     (in_bom yes) (on_board yes) (dnp no)
-    (property "Reference" "R17" (at 127 102.87 90)
+    (property "Reference" "R18" (at 127 102.87 90)
       (effects (font (size 1.27 1.27)))
     )
@@
       (project "USBHUB"
         (path "/d5edc647-9ac3-4ac1-ab8a-57c77be3f4d3/2bd96af5-5a66-4797-badd-32cacbbf4fbd/38e014e7-3281-4b3d-a8ed-ec581f581dff"
-          (reference "R17") (unit 1)
+          (reference "R18") (unit 1)
         )
       )
@@
   (symbol (lib_id "Device:R") (at 152.4 57.15 0) (unit 1)
     (in_bom yes) (on_board yes) (dnp no) (fields_autoplaced)
-    (property "Reference" "R15" (at 154.94 55.88 0)
+    (property "Reference" "R16" (at 154.94 55.88 0)
       (effects (font (size 1.27 1.27)) (justify left))
     )
@@
       (project "USBHUB"
         (path "/d5edc647-9ac3-4ac1-ab8a-57c77be3f4d3/2bd96af5-5a66-4797-badd-32cacbbf4fbd/38e014e7-3281-4b3d-a8ed-ec581f581dff"
-          (reference "R15") (unit 1)
+          (reference "R16") (unit 1)
         )
       )
@@
   (symbol (lib_id "Device:R") (at 152.4 36.83 0) (unit 1)
     (in_bom yes) (on_board yes) (dnp no) (fields_autoplaced)
-    (property "Reference" "R12" (at 154.94 35.56 0)
+    (property "Reference" "R13" (at 154.94 35.56 0)
       (effects (font (size 1.27 1.27)) (justify left))
     )
@@
       (project "USBHUB"
         (path "/d5edc647-9ac3-4ac1-ab8a-57c77be3f4d3/2bd96af5-5a66-4797-badd-32cacbbf4fbd/38e014e7-3281-4b3d-a8ed-ec581f581dff"
-          (reference "R12") (unit 1)
+          (reference "R13") (unit 1)
         )
       )
@@
   (symbol (lib_id "Device:R") (at 115.57 45.72 0) (unit 1)
     (in_bom yes) (on_board yes) (dnp no) (fields_autoplaced)
-    (property "Reference" "R13" (at 118.11 44.45 0)
+    (property "Reference" "R14" (at 118.11 44.45 0)
       (effects (font (size 1.27 1.27)) (justify left))
     )
@@
       (project "USBHUB"
         (path "/d5edc647-9ac3-4ac1-ab8a-57c77be3f4d3/2bd96af5-5a66-4797-badd-32cacbbf4fbd/38e014e7-3281-4b3d-a8ed-ec581f581dff"
-          (reference "R13") (unit 1)
+          (reference "R14") (unit 1)
         )
       )
@@
   (symbol (lib_id "Device:R") (at 138.43 115.57 0) (unit 1)
     (in_bom yes) (on_board yes) (dnp no) (fields_autoplaced)
-    (property "Reference" "R19" (at 140.97 114.3 0)
+    (property "Reference" "R20" (at 140.97 114.3 0)
       (effects (font (size 1.27 1.27)) (justify left))
     )
@@
       (project "USBHUB"
         (path "/d5edc647-9ac3-4ac1-ab8a-57c77be3f4d3/2bd96af5-5a66-4797-badd-32cacbbf4fbd/38e014e7-3281-4b3d-a8ed-ec581f581dff"
-          (reference "R19") (unit 1)
-        )
-      )
+          (reference "R20") (unit 1)
+        )
+      )

Commit message: add schottky for usb pd
Parts:
- D3: value B340 -> Schottky; footprint Diode_SMD:D_SMC -> Diode_SMD:D_SMA
Changed lines of the file:
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@@
       (effects (font (size 1.27 1.27)) (justify left))
     )
-    (property "Value" "B340" (at 106.68 31.4325 90)
+    (property "Value" "Schottky" (at 106.68 31.4325 90)
       (effects (font (size 1.27 1.27)) (justify left))
     )
-    (property "Footprint" "Diode_SMD:D_SMC" (at 99.695 30.48 0)
+    (property "Footprint" "Diode_SMD:D_SMA" (at 99.695 30.48 0)
       (effects (font (size 1.27 1.27)) hide)
     )
-    (property "Datasheet" "http://www.jameco.com/Jameco/Products/ProdDS/1538777.pdf" (at 104.14 30.48 0)
+    (property "Datasheet" "" (at 104.14 30.48 0)
       (effects (font (size 1.27 1.27)) hide)
     )

Commit message: finish layout draft
Connections:
- net GND: now also U3.4 (NC)
Changed lines of the file:
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@@
   (junction (at 191.77 86.36) (diameter 0) (color 0 0 0 0)
+  )
+  (junction (at 217.17 99.06) (diameter 0) (color 0 0 0 0)
   )
   (junction (at 138.43 120.65) (diameter 0) (color 0 0 0 0)
@@
     (stroke (width 0) (type default))
   )
+  (wire (pts (xy 217.17 88.9) (xy 217.17 99.06))
+    (stroke (width 0) (type default))
+  )
   (wire (pts (xy 100.33 113.03) (xy 100.33 115.57))
     (stroke (width 0) (type default))
@@
     (stroke (width 0) (type default))
   )
-  (wire (pts (xy 227.33 99.06) (xy 209.55 99.06))
+  (wire (pts (xy 227.33 99.06) (xy 217.17 99.06))
     (stroke (width 0) (type default))
   )
@@
   )
   (wire (pts (xy 97.79 41.91) (xy 115.57 41.91))
+    (stroke (width 0) (type default))
+  )
+  (wire (pts (xy 217.17 99.06) (xy 209.55 99.06))
     (stroke (width 0) (type default))
   )
@@
       (effects (font (size 1.27 1.27) italic) hide)
     )
-    (property "Datasheet" "https://www.ti.com/lit/ds/symlink/tlv757p.pdf" (at 209.55 87.63 0)
-      (effects (font (size 1.27 1.27)) hide)
-    )
+    (property "Datasheet" "https://www.ti.com/lit/ds/symlink/tlv757p.pdf" (at 209.55 85.09 0)
+      (effects (font (size 1.27 1.27)) hide)
+    )

Commit message: finish bom list
Parts:
- removed D3: Schottky, Diode_SMD:D_SMA, symbol Diode:B340
- added D3: SS54, Diode_SMD:D_SMA, symbol Device:D_Schottky
- C21, C23, C24: footprint Capacitor_SMD:C_0603_1608Metric -> Capacitor_SMD:C_0805_2012Metric
Connections:
- net GND: now also D3.2 (A)
- net at C9.1, L1.1, U2.8 (PH): now also D3.1 (K)
Changed lines of the file:
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@@
-    )
-  )
-  (symbol (lib_id "Diode:B340") (at 104.14 30.48 270) (unit 1)
-    (in_bom yes) (on_board yes) (dnp no) (fields_autoplaced)
-    (property "Reference" "D3" (at 106.68 28.8925 90)
-      (effects (font (size 1.27 1.27)) (justify left))
-    )
-    (property "Value" "Schottky" (at 106.68 31.4325 90)
-      (effects (font (size 1.27 1.27)) (justify left))
-    )
-    (property "Footprint" "Diode_SMD:D_SMA" (at 99.695 30.48 0)
-      (effects (font (size 1.27 1.27)) hide)
-    )
-    (property "Datasheet" "" (at 104.14 30.48 0)
-      (effects (font (size 1.27 1.27)) hide)
-    )
-    (pin "2")
-    (pin "1")
-    (instances
-      (project "USBHUB"
-        (path "/d5edc647-9ac3-4ac1-ab8a-57c77be3f4d3/2bd96af5-5a66-4797-badd-32cacbbf4fbd/38e014e7-3281-4b3d-a8ed-ec581f581dff"
-          (reference "D3") (unit 1)
-        )
-      )
     )
   )
@@
       (effects (font (size 1.27 1.27)) (justify left))
     )
-    (property "Footprint" "Capacitor_SMD:C_0603_1608Metric" (at 158.4452 111.76 0)
+    (property "Footprint" "Capacitor_SMD:C_0805_2012Metric" (at 158.4452 111.76 0)
       (effects (font (size 1.27 1.27)) hide)
     )
@@
       (effects (font (size 1.27 1.27)) (justify left))
     )
-    (property "Footprint" "Capacitor_SMD:C_0603_1608Metric" (at 36.5252 107.95 0)
+    (property "Footprint" "Capacitor_SMD:C_0805_2012Metric" (at 36.5252 107.95 0)
       (effects (font (size 1.27 1.27)) hide)
     )
@@
       (effects (font (size 1.27 1.27)) (justify left))
     )
-    (property "Footprint" "Capacitor_SMD:C_0603_1608Metric" (at 148.2852 111.76 0)
+    (property "Footprint" "Capacitor_SMD:C_0805_2012Metric" (at 148.2852 111.76 0)
       (effects (font (size 1.27 1.27)) hide)
     )
@@
         )
       )
+    )
+  )
+  (symbol (lib_id "Device:D_Schottky") (at 104.14 30.48 270) (unit 1)
+    (in_bom yes) (on_board yes) (dnp no) (fields_autoplaced)
+    (property "Reference" "D3" (at 106.68 28.8925 90)
+      (effects (font (size 1.27 1.27)) (justify left))
+    )
+    (property "Value" "SS54" (at 106.68 31.4325 90)
+      (effects (font (size 1.27 1.27)) (justify left))
+    )
+    (property "Footprint" "Diode_SMD:D_SMA" (at 104.14 30.48 0)
+      (effects (font (size 1.27 1.27)) hide)
+    )
+    (property "Datasheet" "~" (at 104.14 30.48 0)
+      (effects (font (size 1.27 1.27)) hide)
+    )
+    (pin "1")
+    (pin "2")
+    (instances
+      (project "USBHUB"
+        (path "/d5edc647-9ac3-4ac1-ab8a-57c77be3f4d3/2bd96af5-5a66-4797-badd-32cacbbf4fbd/38e014e7-3281-4b3d-a8ed-ec581f581dff"
+          (reference "D3") (unit 1)
+        )
+      )
